Commit message: added rviz

File: rs_description/urdf/spot.urdf.xacro (robot description, xacro)
@@ -2,8 +2,4 @@
 <robot name="spot" xmlns:xacro="http://www.ros.org/wiki/xacro">
     <link name="body">
-    <inertial>
-    <mass value="1.25" />
-    <inertia  ixx="0.1" ixy="0.0"  ixz="0.0"  iyy="0.1"  iyz="0.0"  izz="0.077" />
-    </inertial>
         <visual>
             <geometry>
@@ -16,6 +12,10 @@
             </geometry>
         </collision>
-    </link>
-<link name="base_link"/>
+        <inertial>
+             <mass value="1.25" />
+             <inertia  ixx="0.1" ixy="0.0"  ixz="0.0"  iyy="0.1"  iyz="0.0"  izz="0.077" />
+    	</inertial>
+    </link>
+    <link name="base_link"/>
     <joint name="base_link_joint" type="fixed">
         <origin xyz="0 0 0" rpy="0 0 0" />
@@ -36,8 +36,4 @@
     </joint>
     <link name="front_left_hip">
-        <inertial>
-        <mass value="0.5" />
-    	<inertia  ixx="0.0001" ixy="0.0"  ixz="0.0"  iyy="0.0"  iyz="0.0"  izz="0.0" />
-    	</inertial>
         <visual>
             <geometry>
@@ -50,4 +46,8 @@
             </geometry>
         </collision>
+        <inertial>
+            <mass value="0.5" />
+    	    <inertia  ixx="0.01" ixy="0.0"  ixz="0.0"  iyy="0.0"  iyz="0.0"  izz="0.0" />
+    	</inertial>
     </link>
     <joint name="front_left_hip_x" type="revolute">
@@ -59,8 +59,4 @@
     </joint>
     <link name="front_left_upper_leg">
-        <inertial>
-        <mass value="2.5" />
-    	<inertia  ixx="0.8" ixy="0.0"  ixz="0.0"  iyy="0.2"  iyz="0.0"  izz="0.0" />
-    	</inertial>
         <visual>
             <geometry>
@@ -73,4 +69,8 @@
             </geometry>
         </collision>
+        <inertial>
+            <mass value="2.5" />
+    	    <inertia  ixx="0.8" ixy="0.0"  ixz="0.0"  iyy="0.2"  iyz="0.0"  izz="0.0" />
+    	</inertial>
     </link>
     <joint name="front_left_hip_y" type="revolute">
@@ -82,8 +82,4 @@
     </joint>
     <link name="front_left_lower_leg">
-        <inertial>
-        <mass value="1.5" />
-    	<inertia  ixx="0.0" ixy="0.0"  ixz="0.0"  iyy="0.125"  iyz="0.0"  izz="0.0" />
-    	</inertial>
         <visual>
             <geometry>
@@ -96,4 +92,8 @@
             </geometry>
         </collision>
+        <inertial>
+            <mass value="1.5" />
+    	    <inertia  ixx="0.0" ixy="0.0"  ixz="0.0"  iyy="0.125"  iyz="0.0"  izz="0.0" />
+    	</inertial>
     </link>
     <joint name="front_left_knee" type="revolute">
@@ -105,8 +105,4 @@
     </joint>
     <link name="front_right_hip">
-        <inertial>
-        <mass value="0.5" />
-    	<inertia  ixx="0.0001" ixy="0.0"  ixz="0.0"  iyy="0.0"  iyz="0.0"  izz="0.0" />
-    	</inertial>
         <visual>
             <geometry>
@@ -119,4 +115,8 @@
             </geometry>
         </collision>
+        <inertial>
+            <mass value="0.5" />
+    	    <inertia  ixx="0.01" ixy="0.0"  ixz="0.0"  iyy="0.0"  iyz="0.0"  izz="0.0" />
+    	</inertial>
     </link>
     <joint name="front_right_hip_x" type="revolute">
@@ -128,8 +128,4 @@
     </joint>
     <link name="front_right_upper_leg">
-        <inertial>
-        <mass value="2.5" />
-    	<inertia  ixx="0.8" ixy="0.0"  ixz="0.0"  iyy="0.2"  iyz="0.0"  izz="0.0" />
-    	</inertial>
         <visual>
             <geometry>
@@ -142,4 +138,8 @@
             </geometry>
         </collision>
+        <inertial>
+            <mass value="2.5" />
+    	    <inertia  ixx="0.8" ixy="0.0"  ixz="0.0"  iyy="0.2"  iyz="0.0"  izz="0.0" />
+    	</inertial>
     </link>
     <joint name="front_right_hip_y" type="revolute">
@@ -151,8 +151,4 @@
     </joint>
     <link name="front_right_lower_leg">
-        <inertial>
-        <mass value="1.5" />
-    	<inertia  ixx="0.0" ixy="0.0"  ixz="0.0"  iyy="0.125"  iyz="0.0"  izz="0.0" />
-    	</inertial>
         <visual>
             <geometry>
@@ -165,4 +161,8 @@
             </geometry>
         </collision>
+        <inertial>
+            <mass value="1.5" />
+    	    <inertia  ixx="0.0" ixy="0.0"  ixz="0.0"  iyy="0.125"  iyz="0.0"  izz="0.0" />
+    	</inertial>
     </link>
     <joint name="front_right_knee" type="revolute">
@@ -174,8 +174,4 @@
     </joint>
     <link name="rear_left_hip">
-        <inertial>
-        <mass value="0.5" />
-    	<inertia  ixx="0.0001" ixy="0.0"  ixz="0.0"  iyy="0.0"  iyz="0.0"  izz="0.0" />
-    	</inertial>
         <visual>
             <geometry>
@@ -188,4 +184,8 @@
             </geometry>
         </collision>
+        <inertial>
+            <mass value="0.5" />
+    	    <inertia  ixx="0.01" ixy="0.0"  ixz="0.0"  iyy="0.0"  iyz="0.0"  izz="0.0" />
+    	</inertial>
     </link>
     <joint name="rear_left_hip_x" type="revolute">
@@ -197,8 +197,4 @@
     </joint>
     <link name="rear_left_upper_leg">
-        <inertial>
-        <mass value="2.5" />
-    	<inertia  ixx="0.8" ixy="0.0"  ixz="0.0"  iyy="0.2"  iyz="0.0"  izz="0.0" />
-    	</inertial>
         <visual>
             <geometry>
@@ -211,4 +207,8 @@
             </geometry>
         </collision>
+        <inertial>
+           <mass value="2.5" />
+    	   <inertia  ixx="0.8" ixy="0.0"  ixz="0.0"  iyy="0.2"  iyz="0.0"  izz="0.0" />
+    	</inertial>
     </link>
     <joint name="rear_left_hip_y" type="revolute">
@@ -220,8 +220,4 @@
     </joint>
     <link name="rear_left_lower_leg">
-        <inertial>
-        <mass value="1.5" />
-    	<inertia  ixx="0.0" ixy="0.0"  ixz="0.0"  iyy="0.125"  iyz="0.0"  izz="0.0" />
-    	</inertial>
         <visual>
             <geometry>
@@ -234,4 +230,8 @@
             </geometry>
         </collision>
+        <inertial>
+            <mass value="1.5" />
+    	    <inertia  ixx="0.0" ixy="0.0"  ixz="0.0"  iyy="0.125"  iyz="0.0"  izz="0.0" />
+    	</inertial>
     </link>
     <joint name="rear_left_knee" type="revolute">
@@ -243,8 +243,4 @@
     </joint>
     <link name="rear_right_hip">
-        <inertial>
-        <mass value="0.5" />
-    	<inertia  ixx="0.0001" ixy="0.0"  ixz="0.0"  iyy="0.0"  iyz="0.0"  izz="0.0" />
-    	</inertial>
         <visual>
             <geometry>
@@ -257,4 +253,8 @@
             </geometry>
         </collision>
+        <inertial>
+            <mass value="0.5" />
+    	    <inertia  ixx="0.01" ixy="0.0"  ixz="0.0"  iyy="0.0"  iyz="0.0"  izz="0.0" />
+    	</inertial>
     </link>
     <joint name="rear_right_hip_x" type="revolute">
@@ -266,8 +266,4 @@
     </joint>
     <link name="rear_right_upper_leg">
-        <inertial>
-        <mass value="2.5" />
-    	<inertia  ixx="0.8" ixy="0.0"  ixz="0.0"  iyy="0.2"  iyz="0.0"  izz="0.0" />
-    	</inertial>
         <visual>
             <geometry>
@@ -280,4 +276,8 @@
             </geometry>
         </collision>
+        <inertial>
+            <mass value="2.5" />
+    	    <inertia  ixx="0.8" ixy="0.0"  ixz="0.0"  iyy="0.2"  iyz="0.0"  izz="0.0" />
+    	</inertial>
     </link>
     <joint name="rear_right_hip_y" type="revolute">
@@ -289,8 +289,4 @@
     </joint>
     <link name="rear_right_lower_leg">
-        <inertial>
-        <mass value="1.5" />
-    	<inertia  ixx="0.0" ixy="0.0"  ixz="0.0"  iyy="0.125"  iyz="0.0"  izz="0.0" />
-    	</inertial>
         <visual>
             <geometry>
@@ -303,4 +299,8 @@
             </geometry>
         </collision>
+        <inertial>
+            <mass value="1.5" />
+    	    <inertia  ixx="0.0" ixy="0.0"  ixz="0.0"  iyy="0.125"  iyz="0.0"  izz="0.0" />
+    	</inertial>
     </link>
     <joint name="rear_right_knee" type="revolute">
@@ -311,3 +311,5 @@
         <limit effort="1000" velocity="1000.00" lower="-2.7929" upper="-0.257725" />
     </joint>
+    <!-- Optional custom includes. -->
+    <xacro:include filename="$(optenv SPOT_URDF_EXTRAS empty.urdf)" />
 </robot>

Commit message: joint plugin

File: rs_description/urdf/spot.urdf.xacro (robot description, xacro)
@@ -4,10 +4,10 @@
         <visual>
             <geometry>
-                <mesh filename="package://spot_description/meshes/body.dae" />
-            </geometry>
-        </visual>
-        <collision>
-            <geometry>
-                <mesh filename="package://spot_description/meshes/body_collision.stl" />
+                <mesh filename="package://rs_description/meshes/body.dae" />
+            </geometry>
+        </visual>
+        <collision>
+            <geometry>
+                <mesh filename="package://rs_description/meshes/body_collision.stl" />
             </geometry>
         </collision>
@@ -38,10 +38,10 @@
         <visual>
             <geometry>
-                <mesh filename="package://spot_description/meshes/front_left_hip.dae" />
-            </geometry>
-        </visual>
-        <collision>
-            <geometry>
-                <mesh filename="package://spot_description/meshes/front_left_hip_collision.stl" />
+                <mesh filename="package://rs_description/meshes/front_left_hip.dae" />
+            </geometry>
+        </visual>
+        <collision>
+            <geometry>
+                <mesh filename="package://rs_description/meshes/front_left_hip_collision.stl" />
             </geometry>
         </collision>
@@ -61,10 +61,10 @@
         <visual>
             <geometry>
-                <mesh filename="package://spot_description/meshes/front_left_upper_leg.dae" />
-            </geometry>
-        </visual>
-        <collision>
-            <geometry>
-                <mesh filename="package://spot_description/meshes/front_left_upper_leg_collision.stl" />
+                <mesh filename="package://rs_description/meshes/front_left_upper_leg.dae" />
+            </geometry>
+        </visual>
+        <collision>
+            <geometry>
+                <mesh filename="package://rs_description/meshes/front_left_upper_leg_collision.stl" />
             </geometry>
         </collision>
@@ -84,10 +84,10 @@
         <visual>
             <geometry>
-                <mesh filename="package://spot_description/meshes/front_left_lower_leg.dae" />
-            </geometry>
-        </visual>
-        <collision>
-            <geometry>
-                <mesh filename="package://spot_description/meshes/front_left_lower_leg_collision.stl" />
+                <mesh filename="package://rs_description/meshes/front_left_lower_leg.dae" />
+            </geometry>
+        </visual>
+        <collision>
+            <geometry>
+                <mesh filename="package://rs_description/meshes/front_left_lower_leg_collision.stl" />
             </geometry>
         </collision>
@@ -107,10 +107,10 @@
         <visual>
             <geometry>
-                <mesh filename="package://spot_description/meshes/front_right_hip.dae" />
-            </geometry>
-        </visual>
-        <collision>
-            <geometry>
-                <mesh filename="package://spot_description/meshes/front_right_hip_collision.stl" />
+                <mesh filename="package://rs_description/meshes/front_right_hip.dae" />
+            </geometry>
+        </visual>
+        <collision>
+            <geometry>
+                <mesh filename="package://rs_description/meshes/front_right_hip_collision.stl" />
             </geometry>
         </collision>
@@ -130,10 +130,10 @@
         <visual>
             <geometry>
-                <mesh filename="package://spot_description/meshes/front_right_upper_leg.dae" />
-            </geometry>
-        </visual>
-        <collision>
-            <geometry>
-                <mesh filename="package://spot_description/meshes/front_right_upper_leg_collision.stl" />
+                <mesh filename="package://rs_description/meshes/front_right_upper_leg.dae" />
+            </geometry>
+        </visual>
+        <collision>
+            <geometry>
+                <mesh filename="package://rs_description/meshes/front_right_upper_leg_collision.stl" />
             </geometry>
         </collision>
@@ -153,10 +153,10 @@
         <visual>
             <geometry>
-                <mesh filename="package://spot_description/meshes/front_right_lower_leg.dae" />
-            </geometry>
-        </visual>
-        <collision>
-            <geometry>
-                <mesh filename="package://spot_description/meshes/front_right_lower_leg_collision.stl" />
+                <mesh filename="package://rs_description/meshes/front_right_lower_leg.dae" />
+            </geometry>
+        </visual>
+        <collision>
+            <geometry>
+                <mesh filename="package://rs_description/meshes/front_right_lower_leg_collision.stl" />
             </geometry>
         </collision>
@@ -176,10 +176,10 @@
         <visual>
             <geometry>
-                <mesh filename="package://spot_description/meshes/rear_left_hip.dae" />
-            </geometry>
-        </visual>
-        <collision>
-            <geometry>
-                <mesh filename="package://spot_description/meshes/rear_left_hip_collision.stl" />
+                <mesh filename="package://rs_description/meshes/rear_left_hip.dae" />
+            </geometry>
+        </visual>
+        <collision>
+            <geometry>
+                <mesh filename="package://rs_description/meshes/rear_left_hip_collision.stl" />
             </geometry>
         </collision>
@@ -199,10 +199,10 @@
         <visual>
             <geometry>
-                <mesh filename="package://spot_description/meshes/rear_left_upper_leg.dae" />
-            </geometry>
-        </visual>
-        <collision>
-            <geometry>
-                <mesh filename="package://spot_description/meshes/rear_left_upper_leg_collision.stl" />
+                <mesh filename="package://rs_description/meshes/rear_left_upper_leg.dae" />
+            </geometry>
+        </visual>
+        <collision>
+            <geometry>
+                <mesh filename="package://rs_description/meshes/rear_left_upper_leg_collision.stl" />
             </geometry>
         </collision>
@@ -222,10 +222,10 @@
         <visual>
             <geometry>
-                <mesh filename="package://spot_description/meshes/rear_left_lower_leg.dae" />
-            </geometry>
-        </visual>
-        <collision>
-            <geometry>
-                <mesh filename="package://spot_description/meshes/rear_left_lower_leg_collision.stl" />
+                <mesh filename="package://rs_description/meshes/rear_left_lower_leg.dae" />
+            </geometry>
+        </visual>
+        <collision>
+            <geometry>
+                <mesh filename="package://rs_description/meshes/rear_left_lower_leg_collision.stl" />
             </geometry>
         </collision>
@@ -245,10 +245,10 @@
         <visual>
             <geometry>
-                <mesh filename="package://spot_description/meshes/rear_right_hip.dae" />
-            </geometry>
-        </visual>
-        <collision>
-            <geometry>
-                <mesh filename="package://spot_description/meshes/rear_right_hip_collision.stl" />
+                <mesh filename="package://rs_description/meshes/rear_right_hip.dae" />
+            </geometry>
+        </visual>
+        <collision>
+            <geometry>
+                <mesh filename="package://rs_description/meshes/rear_right_hip_collision.stl" />
             </geometry>
         </collision>
@@ -268,10 +268,10 @@
         <visual>
             <geometry>
-                <mesh filename="package://spot_description/meshes/rear_right_upper_leg.dae" />
-            </geometry>
-        </visual>
-        <collision>
-            <geometry>
-                <mesh filename="package://spot_description/meshes/rear_right_upper_leg_collision.stl" />
+                <mesh filename="package://rs_description/meshes/rear_right_upper_leg.dae" />
+            </geometry>
+        </visual>
+        <collision>
+            <geometry>
+                <mesh filename="package://rs_description/meshes/rear_right_upper_leg_collision.stl" />
             </geometry>
         </collision>
@@ -291,10 +291,10 @@
         <visual>
             <geometry>
-                <mesh filename="package://spot_description/meshes/rear_right_lower_leg.dae" />
-            </geometry>
-        </visual>
-        <collision>
-            <geometry>
-                <mesh filename="package://spot_description/meshes/rear_right_lower_leg_collision.stl" />
+                <mesh filename="package://rs_description/meshes/rear_right_lower_leg.dae" />
+            </geometry>
+        </visual>
+        <collision>
+            <geometry>
+                <mesh filename="package://rs_description/meshes/rear_right_lower_leg_collision.stl" />
             </geometry>
         </collision>
@@ -311,4 +311,17 @@
         <limit effort="1000" velocity="1000.00" lower="-2.7929" upper="-0.257725" />
     </joint>
+    <!--Publish joint state from Gazebo-->
+        <plugin name="joint_state_publisher" filename="libgazebo_ros_joint_state_publisher.so">
+            <robotNamespace>robot</robotNamespace>
+            <jointName>
+                base_link_joint, front_rail_joint, rear_rail_joint,
+                front_left_hip_x, front_left_hip_y, front_left_knee,
+                front_right_hip_x, front_right_hip_y, front_right_knee,
+                rear_left_hip_x, rear_left_hip_y, rear_left_knee,
+                rear_right_hip_x, rear_right_hip_y, rear_right_knee
+            </jointName>
+            <updateRate>100</updateRate>
+            <alwaysOn>true</alwaysOn>
+        </plugin>
     <!-- Optional custom includes. -->
     <xacro:include filename="$(optenv SPOT_URDF_EXTRAS empty.urdf)" />
