Commit message: tf_fixes

File: rs_description/urdf/spot.urdf.xacro (robot description, xacro)
@@ -55,7 +55,18 @@
         <axis xyz="1 0 0" />
         <parent link="body" />
-        <child link="front_left_hip" />
+	<child link="front_left_hip" />
+	<dynamics damping="0.0" friction="0.0"/>
         <limit effort="1000" velocity="1000.00" lower="-0.78539816339744827899" upper="0.78539816339744827899" />
-    </joint>
+</joint>
+<transmission name="simple_trans">
+	  <type>transmission_interface/SimpleTransmission</type>
+	    <joint name="front_left_hip_x">
+		        <hardwareInterface>EffortJointInterface</hardwareInterface>
+			  </joint>
+			    <actuator name="front_left_hip_x">
+				        <mechanicalReduction>50</mechanicalReduction>
+					    <hardwareInterface>EffortJointInterface</hardwareInterface>
+					      </actuator>
+				      </transmission>
     <link name="front_left_upper_leg">
         <visual>
@@ -78,5 +89,6 @@
         <axis xyz="0 1 0" />
         <parent link="front_left_hip" />
-        <child link="front_left_upper_leg" />
+	<child link="front_left_upper_leg" />
+	<dynamics damping="0.0" friction="0.0"/>
         <limit effort="1000" velocity="1000.00" lower="-0.89884456477707963539" upper="2.2951079663725435509" />
     </joint>
@@ -103,226 +115,17 @@
         <child link="front_left_lower_leg" />
         <limit effort="1000" velocity="1000.00" lower="-2.7929" upper="-0.254801" />
-    </joint>
-    <link name="front_right_hip">
-        <visual>
-            <geometry>
-                <mesh filename="package://rs_description/meshes/front_right_hip.dae" />
-            </geometry>
-        </visual>
-        <collision>
-            <geometry>
-                <mesh filename="package://rs_description/meshes/front_right_hip_collision.stl" />
-            </geometry>
-        </collision>
-        <inertial>
-            <mass value="0.5" />
-    	    <inertia  ixx="0.01" ixy="0.0"  ixz="0.0"  iyy="0.0"  iyz="0.0"  izz="0.0" />
-    	</inertial>
-    </link>
-    <joint name="front_right_hip_x" type="revolute">
-        <origin xyz="0.29785 -0.05500 0.00000" rpy="0 0 0" />
-        <axis xyz="1 0 0" />
-        <parent link="body" />
-        <child link="front_right_hip" />
-        <limit effort="1000" velocity="1000.00" lower="-0.78539816339744827899" upper="0.78539816339744827899" />
-    </joint>
-    <link name="front_right_upper_leg">
-        <visual>
-            <geometry>
-                <mesh filename="package://rs_description/meshes/front_right_upper_leg.dae" />
-            </geometry>
-        </visual>
-        <collision>
-            <geometry>
-                <mesh filename="package://rs_description/meshes/front_right_upper_leg_collision.stl" />
-            </geometry>
-        </collision>
-        <inertial>
-            <mass value="2.5" />
-    	    <inertia  ixx="0.8" ixy="0.0"  ixz="0.0"  iyy="0.2"  iyz="0.0"  izz="0.0" />
-    	</inertial>
-    </link>
-    <joint name="front_right_hip_y" type="revolute">
-        <origin xyz="0.0 -0.110945 0.0" rpy="0 0 0" />
-        <axis xyz="0 1 0" />
-        <parent link="front_right_hip" />
-        <child link="front_right_upper_leg" />
-        <limit effort="1000" velocity="1000.00" lower="-0.89884456477707963539" upper="2.2951079663725435509" />
-    </joint>
-    <link name="front_right_lower_leg">
-        <visual>
-            <geometry>
-                <mesh filename="package://rs_description/meshes/front_right_lower_leg.dae" />
-            </geometry>
-        </visual>
-        <collision>
-            <geometry>
-                <mesh filename="package://rs_description/meshes/front_right_lower_leg_collision.stl" />
-            </geometry>
-        </collision>
-        <inertial>
-            <mass value="1.5" />
-    	    <inertia  ixx="0.0" ixy="0.0"  ixz="0.0"  iyy="0.125"  iyz="0.0"  izz="0.0" />
-    	</inertial>
-    </link>
-    <joint name="front_right_knee" type="revolute">
-        <origin xyz="0.025 0.000 -0.3205" rpy="0 0 0" />
-        <axis xyz="0 1 0" />
-        <parent link="front_right_upper_leg" />
-        <child link="front_right_lower_leg" />
-        <limit effort="1000" velocity="1000.00" lower="-2.7929" upper="-0.247563" />
-    </joint>
-    <link name="rear_left_hip">
-        <visual>
-            <geometry>
-                <mesh filename="package://rs_description/meshes/rear_left_hip.dae" />
-            </geometry>
-        </visual>
-        <collision>
-            <geometry>
-                <mesh filename="package://rs_description/meshes/rear_left_hip_collision.stl" />
-            </geometry>
-        </collision>
-        <inertial>
-            <mass value="0.5" />
-    	    <inertia  ixx="0.01" ixy="0.0"  ixz="0.0"  iyy="0.0"  iyz="0.0"  izz="0.0" />
-    	</inertial>
-    </link>
-    <joint name="rear_left_hip_x" type="revolute">
-        <origin xyz="-0.29785 0.05500 0.00000" rpy="0 0 0" />
-        <axis xyz="1 0 0" />
-        <parent link="body" />
-        <child link="rear_left_hip" />
-        <limit effort="1000" velocity="1000.00" lower="-0.78539816339744827899" upper="0.78539816339744827899" />
-    </joint>
-    <link name="rear_left_upper_leg">
-        <visual>
-            <geometry>
-                <mesh filename="package://rs_description/meshes/rear_left_upper_leg.dae" />
-            </geometry>
-        </visual>
-        <collision>
-            <geometry>
-                <mesh filename="package://rs_description/meshes/rear_left_upper_leg_collision.stl" />
-            </geometry>
-        </collision>
-        <inertial>
-           <mass value="2.5" />
-    	   <inertia  ixx="0.8" ixy="0.0"  ixz="0.0"  iyy="0.2"  iyz="0.0"  izz="0.0" />
-    	</inertial>
-    </link>
-    <joint name="rear_left_hip_y" type="revolute">
-        <origin xyz="0.0 0.110945 0.0" rpy="0 0 0" />
-        <axis xyz="0 1 0" />
-        <parent link="rear_left_hip" />
-        <child link="rear_left_upper_leg" />
-        <limit effort="1000" velocity="1000.00" lower="-0.89884456477707963539" upper="2.2951079663725435509" />
-    </joint>
-    <link name="rear_left_lower_leg">
-        <visual>
-            <geometry>
-                <mesh filename="package://rs_description/meshes/rear_left_lower_leg.dae" />
-            </geometry>
-        </visual>
-        <collision>
-            <geometry>
-                <mesh filename="package://rs_description/meshes/rear_left_lower_leg_collision.stl" />
-            </geometry>
-        </collision>
-        <inertial>
-            <mass value="1.5" />
-    	    <inertia  ixx="0.0" ixy="0.0"  ixz="0.0"  iyy="0.125"  iyz="0.0"  izz="0.0" />
-    	</inertial>
-    </link>
-    <joint name="rear_left_knee" type="revolute">
-        <origin xyz="0.025 0.000 -0.3205" rpy="0 0 0" />
-        <axis xyz="0 1 0" />
-        <parent link="rear_left_upper_leg" />
-        <child link="rear_left_lower_leg" />
-        <limit effort="1000" velocity="1000.00" lower="-2.7929" upper="-0.267153" />
-    </joint>
-    <link name="rear_right_hip">
-        <visual>
-            <geometry>
-                <mesh filename="package://rs_description/meshes/rear_right_hip.dae" />
-            </geometry>
-        </visual>
-        <collision>
-            <geometry>
-                <mesh filename="package://rs_description/meshes/rear_right_hip_collision.stl" />
-            </geometry>
-        </collision>
-        <inertial>
-            <mass value="0.5" />
-    	    <inertia  ixx="0.01" ixy="0.0"  ixz="0.0"  iyy="0.0"  iyz="0.0"  izz="0.0" />
-    	</inertial>
-    </link>
-    <joint name="rear_right_hip_x" type="revolute">
-        <origin xyz="-0.29785 -0.05500 0.00000" rpy="0 0 0" />
-        <axis xyz="1 0 0" />
-        <parent link="body" />
-        <child link="rear_right_hip" />
-        <limit effort="1000" velocity="1000.00" lower="-0.78539816339744827899" upper="0.78539816339744827899" />
-    </joint>
-    <link name="rear_right_upper_leg">
-        <visual>
-            <geometry>
-                <mesh filename="package://rs_description/meshes/rear_right_upper_leg.dae" />
-            </geometry>
-        </visual>
-        <collision>
-            <geometry>
-                <mesh filename="package://rs_description/meshes/rear_right_upper_leg_collision.stl" />
-            </geometry>
-        </collision>
-        <inertial>
-            <mass value="2.5" />
-    	    <inertia  ixx="0.8" ixy="0.0"  ixz="0.0"  iyy="0.2"  iyz="0.0"  izz="0.0" />
-    	</inertial>
-    </link>
-    <joint name="rear_right_hip_y" type="revolute">
-        <origin xyz="0.0 -0.110945 0.0" rpy="0 0 0" />
-        <axis xyz="0 1 0" />
-        <parent link="rear_right_hip" />
-        <child link="rear_right_upper_leg" />
-        <limit effort="1000" velocity="1000.00" lower="-0.89884456477707963539" upper="2.2951079663725435509" />
-    </joint>
-    <link name="rear_right_lower_leg">
-        <visual>
-            <geometry>
-                <mesh filename="package://rs_description/meshes/rear_right_lower_leg.dae" />
-            </geometry>
-        </visual>
-        <collision>
-            <geometry>
-                <mesh filename="package://rs_description/meshes/rear_right_lower_leg_collision.stl" />
-            </geometry>
-        </collision>
-        <inertial>
-            <mass value="1.5" />
-    	    <inertia  ixx="0.0" ixy="0.0"  ixz="0.0"  iyy="0.125"  iyz="0.0"  izz="0.0" />
-    	</inertial>
-    </link>
-    <joint name="rear_right_knee" type="revolute">
-        <origin xyz="0.025 0.000 -0.3205" rpy="0 0 0" />
-        <axis xyz="0 1 0" />
-        <parent link="rear_right_upper_leg" />
-        <child link="rear_right_lower_leg" />
-        <limit effort="1000" velocity="1000.00" lower="-2.7929" upper="-0.257725" />
-    </joint>
+</joint>
     <!--Publish joint state from Gazebo-->
-        <plugin name="joint_state_publisher" filename="libgazebo_ros_joint_state_publisher.so">
-            <robotNamespace>robot</robotNamespace>
-            <jointName>
-                base_link_joint, front_rail_joint, rear_rail_joint,
-                front_left_hip_x, front_left_hip_y, front_left_knee,
-                front_right_hip_x, front_right_hip_y, front_right_knee,
-                rear_left_hip_x, rear_left_hip_y, rear_left_knee,
-                rear_right_hip_x, rear_right_hip_y, rear_right_knee
-            </jointName>
-            <updateRate>100</updateRate>
-            <alwaysOn>true</alwaysOn>
-        </plugin>
-    <!-- Optional custom includes. -->
-    <xacro:include filename="$(optenv SPOT_URDF_EXTRAS empty.urdf)" />
-</robot>
+    <!--            <plugin name="joint_state_publisher" filename="libgazebo_ros_joint_state_publisher.so">
+		                <jointName>
+					                base_link_joint, front_rail_joint, rear_rail_joint,
+							                front_left_hip_x, front_left_hip_y, front_left_knee,
+									                front_right_hip_x, front_right_hip_y, front_right_knee,
+											                rear_left_hip_x, rear_left_hip_y, rear_left_knee,
+													                rear_right_hip_x, rear_right_hip_y, rear_right_knee
+															            </jointName>
+																                <updateRate>100</updateRate>
+																		            <alwaysOn>true</alwaysOn>
+																			            </plugin>
+-->
+																			    </robot>
