Commit message: added translations for all joints

File: rs_description/urdf/spot.urdf.xacro (robot description, xacro)
@@ -1,4 +1,5 @@
 <?xml version="1.0" ?>
 <robot name="spot" xmlns:xacro="http://www.ros.org/wiki/xacro">
+<!-- Body -->
     <link name="body">
         <visual>
@@ -17,4 +18,5 @@
     	</inertial>
     </link>
+<!-- Base link -->
     <link name="base_link"/>
     <joint name="base_link_joint" type="fixed">
@@ -23,4 +25,5 @@
         <child link="base_link" />
     </joint>
+<!-- Front rail -->
     <link name="front_rail"/>
     <joint name="front_rail_joint" type="fixed">
@@ -29,4 +32,5 @@
         <child link="front_rail" />
     </joint>
+<!-- Rear rail -->
     <link name="rear_rail"/>
     <joint name="rear_rail_joint" type="fixed">
@@ -35,4 +39,5 @@
         <child link="rear_rail" />
     </joint>
+<!-- front_left_hip -->
     <link name="front_left_hip">
         <visual>
@@ -58,15 +63,16 @@
 	<dynamics damping="0.0" friction="0.0"/>
         <limit effort="1000" velocity="1000.00" lower="-0.78539816339744827899" upper="0.78539816339744827899" />
-</joint>
-<transmission name="simple_trans">
-	  <type>transmission_interface/SimpleTransmission</type>
-	    <joint name="front_left_hip_x">
-		        <hardwareInterface>EffortJointInterface</hardwareInterface>
-			  </joint>
-			    <actuator name="front_left_hip_x">
-				        <mechanicalReduction>50</mechanicalReduction>
-					    <hardwareInterface>EffortJointInterface</hardwareInterface>
-					      </actuator>
-				      </transmission>
+    </joint>
+    <transmission name="front_left_hip_x_trans">
+	  <type>transmission_interface/SimpleTransmission</type>
+	  <joint name="front_left_hip_x">
+          	<hardwareInterface>EffortJointInterface</hardwareInterface>
+          </joint>
+	  <actuator name="front_left_hip_x">
+          	<mechanicalReduction>50</mechanicalReduction>
+          	<hardwareInterface>EffortJointInterface</hardwareInterface>
+	  </actuator>
+    </transmission>
+<!-- front_left_upper_leg -->
     <link name="front_left_upper_leg">
         <visual>
@@ -93,4 +99,15 @@
         <limit effort="1000" velocity="1000.00" lower="-0.89884456477707963539" upper="2.2951079663725435509" />
     </joint>
+    <transmission name="front_left_hip_y_trans">
+	  <type>transmission_interface/SimpleTransmission</type>
+	  <joint name="front_left_hip_y">
+          	<hardwareInterface>EffortJointInterface</hardwareInterface>
+          </joint>
+	  <actuator name="front_left_hip_y">
+          	<mechanicalReduction>50</mechanicalReduction>
+          	<hardwareInterface>EffortJointInterface</hardwareInterface>
+	  </actuator>
+    </transmission>
+<!-- front_left_lower_leg -->
     <link name="front_left_lower_leg">
         <visual>
@@ -114,18 +131,331 @@
         <parent link="front_left_upper_leg" />
         <child link="front_left_lower_leg" />
+        <dynamics damping="0.0" friction="0.0"/>
         <limit effort="1000" velocity="1000.00" lower="-2.7929" upper="-0.254801" />
-</joint>
-    <!--Publish joint state from Gazebo-->
-    <!--            <plugin name="joint_state_publisher" filename="libgazebo_ros_joint_state_publisher.so">
-		                <jointName>
-					                base_link_joint, front_rail_joint, rear_rail_joint,
-							                front_left_hip_x, front_left_hip_y, front_left_knee,
-									                front_right_hip_x, front_right_hip_y, front_right_knee,
-											                rear_left_hip_x, rear_left_hip_y, rear_left_knee,
-													                rear_right_hip_x, rear_right_hip_y, rear_right_knee
-															            </jointName>
-																                <updateRate>100</updateRate>
-																		            <alwaysOn>true</alwaysOn>
-																			            </plugin>
--->
-																			    </robot>
+    </joint>
+    <transmission name="front_left_knee_trans">
+	  <type>transmission_interface/SimpleTransmission</type>
+	  <joint name="front_left_knee">
+          	<hardwareInterface>EffortJointInterface</hardwareInterface>
+          </joint>
+	  <actuator name="front_left_knee">
+          	<mechanicalReduction>50</mechanicalReduction>
+          	<hardwareInterface>EffortJointInterface</hardwareInterface>
+	  </actuator>
+    </transmission>
+<!--front_right_hip-->
+    <link name="front_right_hip">
+        <visual>
+            <geometry>
+                <mesh filename="package://rs_description/meshes/front_right_hip.dae" />
+            </geometry>
+        </visual>
+        <collision>
+            <geometry>
+                <mesh filename="package://rs_description/meshes/front_right_hip_collision.stl" />
+            </geometry>
+        </collision>
+        <inertial>
+            <mass value="0.5" />
+    	    <inertia  ixx="0.01" ixy="0.0"  ixz="0.0"  iyy="0.0"  iyz="0.0"  izz="0.0" />
+    	</inertial>
+    </link>
+    <joint name="front_right_hip_x" type="revolute">
+        <origin xyz="0.29785 -0.05500 0.00000" rpy="0 0 0" />
+        <axis xyz="1 0 0" />
+        <parent link="body" />
+        <child link="front_right_hip" />
+        <dynamics damping="0.0" friction="0.0"/>
+        <limit effort="1000" velocity="1000.00" lower="-0.78539816339744827899" upper="0.78539816339744827899" />
+    </joint>
+    <transmission name="front_right_hip_x_trans">
+	  <type>transmission_interface/SimpleTransmission</type>
+	  <joint name="front_right_hip_x">
+          	<hardwareInterface>EffortJointInterface</hardwareInterface>
+          </joint>
+	  <actuator name="front_right_hip_x">
+          	<mechanicalReduction>50</mechanicalReduction>
+          	<hardwareInterface>EffortJointInterface</hardwareInterface>
+	  </actuator>
+    </transmission>
+<!-- front_right_upper_leg -->
+    <link name="front_right_upper_leg">
+        <visual>
+            <geometry>
+                <mesh filename="package://rs_description/meshes/front_right_upper_leg.dae" />
+            </geometry>
+        </visual>
+        <collision>
+            <geometry>
+                <mesh filename="package://rs_description/meshes/front_right_upper_leg_collision.stl" />
+            </geometry>
+        </collision>
+        <inertial>
+            <mass value="2.5" />
+    	    <inertia  ixx="0.8" ixy="0.0"  ixz="0.0"  iyy="0.2"  iyz="0.0"  izz="0.0" />
+    	</inertial>
+    </link>
+    <joint name="front_right_hip_y" type="revolute">
+        <origin xyz="0.0 -0.110945 0.0" rpy="0 0 0" />
+        <axis xyz="0 1 0" />
+        <parent link="front_right_hip" />
+        <child link="front_right_upper_leg" />
+        <dynamics damping="0.0" friction="0.0"/>
+        <limit effort="1000" velocity="1000.00" lower="-0.89884456477707963539" upper="2.2951079663725435509" />
+    </joint>
+    <transmission name="front_right_hip_y_trans">
+	  <type>transmission_interface/SimpleTransmission</type>
+	  <joint name="front_right_hip_y">
+          	<hardwareInterface>EffortJointInterface</hardwareInterface>
+          </joint>
+	  <actuator name="front_right_hip_y">
+          	<mechanicalReduction>50</mechanicalReduction>
+          	<hardwareInterface>EffortJointInterface</hardwareInterface>
+	  </actuator>
+    </transmission>
+<!-- front_right_lower_leg -->
+    <link name="front_right_lower_leg">
+        <visual>
+            <geometry>
+                <mesh filename="package://rs_description/meshes/front_right_lower_leg.dae" />
+            </geometry>
+        </visual>
+        <collision>
+            <geometry>
+                <mesh filename="package://rs_description/meshes/front_right_lower_leg_collision.stl" />
+            </geometry>
+        </collision>
+        <inertial>
+            <mass value="1.5" />
+    	    <inertia  ixx="0.0" ixy="0.0"  ixz="0.0"  iyy="0.125"  iyz="0.0"  izz="0.0" />
+    	</inertial>
+    </link>
+    <joint name="front_right_knee" type="revolute">
+        <origin xyz="0.025 0.000 -0.3205" rpy="0 0 0" />
+        <axis xyz="0 1 0" />
+        <parent link="front_right_upper_leg" />
+        <child link="front_right_lower_leg" />
+        <dynamics damping="0.0" friction="0.0"/>
+        <limit effort="1000" velocity="1000.00" lower="-2.7929" upper="-0.247563" />
+    </joint>
+    <transmission name="front_right_knee_trans">
+	  <type>transmission_interface/SimpleTransmission</type>
+	  <joint name="front_right_knee">
+          	<hardwareInterface>EffortJointInterface</hardwareInterface>
+          </joint>
+	  <actuator name="front_right_knee">
+          	<mechanicalReduction>50</mechanicalReduction>
+          	<hardwareInterface>EffortJointInterface</hardwareInterface>
+	  </actuator>
+    </transmission>
+<!-- rear_left_hip -->
+   <link name="rear_left_hip">
+        <visual>
+            <geometry>
+                <mesh filename="package://rs_description/meshes/rear_left_hip.dae" />
+            </geometry>
+        </visual>
+        <collision>
+            <geometry>
+                <mesh filename="package://rs_description/meshes/rear_left_hip_collision.stl" />
+            </geometry>
+        </collision>
+        <inertial>
+            <mass value="0.5" />
+    	    <inertia  ixx="0.01" ixy="0.0"  ixz="0.0"  iyy="0.0"  iyz="0.0"  izz="0.0" />
+    	</inertial>
+    </link>
+    <joint name="rear_left_hip_x" type="revolute">
+        <origin xyz="-0.29785 0.05500 0.00000" rpy="0 0 0" />
+        <axis xyz="1 0 0" />
+        <parent link="body" />
+        <child link="rear_left_hip" />
+        <dynamics damping="0.0" friction="0.0"/>
+        <limit effort="1000" velocity="1000.00" lower="-0.78539816339744827899" upper="0.78539816339744827899" />
+    </joint>
+    <transmission name="rear_left_hip_x_trans">
+	  <type>transmission_interface/SimpleTransmission</type>
+	  <joint name="rear_left_hip_x">
+          	<hardwareInterface>EffortJointInterface</hardwareInterface>
+          </joint>
+	  <actuator name="rear_left_hip_x">
+          	<mechanicalReduction>50</mechanicalReduction>
+          	<hardwareInterface>EffortJointInterface</hardwareInterface>
+	  </actuator>
+    </transmission>
+<!-- rear_left_upper_leg -->
+    <link name="rear_left_upper_leg">
+        <visual>
+            <geometry>
+                <mesh filename="package://rs_description/meshes/rear_left_upper_leg.dae" />
+            </geometry>
+        </visual>
+        <collision>
+            <geometry>
+                <mesh filename="package://rs_description/meshes/rear_left_upper_leg_collision.stl" />
+            </geometry>
+        </collision>
+        <inertial>
+           <mass value="2.5" />
+    	   <inertia  ixx="0.8" ixy="0.0"  ixz="0.0"  iyy="0.2"  iyz="0.0"  izz="0.0" />
+    	</inertial>
+    </link>
+    <joint name="rear_left_hip_y" type="revolute">
+        <origin xyz="0.0 0.110945 0.0" rpy="0 0 0" />
+        <axis xyz="0 1 0" />
+        <parent link="rear_left_hip" />
+        <child link="rear_left_upper_leg" />
+        <dynamics damping="0.0" friction="0.0"/>
+        <limit effort="1000" velocity="1000.00" lower="-0.89884456477707963539" upper="2.2951079663725435509" />
+    </joint>
+    <transmission name="rear_left_hip_y_trans">
+	  <type>transmission_interface/SimpleTransmission</type>
+	  <joint name="rear_left_hip_y">
+          	<hardwareInterface>EffortJointInterface</hardwareInterface>
+          </joint>
+	  <actuator name="rear_left_hip_y">
+          	<mechanicalReduction>50</mechanicalReduction>
+          	<hardwareInterface>EffortJointInterface</hardwareInterface>
+	  </actuator>
+    </transmission>
+<!-- rear_left_lower_leg -->
+    <link name="rear_left_lower_leg">
+        <visual>
+            <geometry>
+                <mesh filename="package://rs_description/meshes/rear_left_lower_leg.dae" />
+            </geometry>
+        </visual>
+        <collision>
+            <geometry>
+                <mesh filename="package://rs_description/meshes/rear_left_lower_leg_collision.stl" />
+            </geometry>
+        </collision>
+        <inertial>
+            <mass value="1.5" />
+    	    <inertia  ixx="0.0" ixy="0.0"  ixz="0.0"  iyy="0.125"  iyz="0.0"  izz="0.0" />
+    	</inertial>
+    </link>
+    <joint name="rear_left_knee" type="revolute">
+        <origin xyz="0.025 0.000 -0.3205" rpy="0 0 0" />
+        <axis xyz="0 1 0" />
+        <parent link="rear_left_upper_leg" />
+        <child link="rear_left_lower_leg" />
+        <dynamics damping="0.0" friction="0.0"/>
+        <limit effort="1000" velocity="1000.00" lower="-2.7929" upper="-0.267153" />
+    </joint>
+    <transmission name="rear_left_knee_trans">
+	  <type>transmission_interface/SimpleTransmission</type>
+	  <joint name="rear_left_knee">
+          	<hardwareInterface>EffortJointInterface</hardwareInterface>
+          </joint>
+	  <actuator name="rear_left_knee">
+          	<mechanicalReduction>50</mechanicalReduction>
+          	<hardwareInterface>EffortJointInterface</hardwareInterface>
+	  </actuator>
+    </transmission>
+<!-- rear_right_hip -->
+   <link name="rear_right_hip">
+        <visual>
+            <geometry>
+                <mesh filename="package://rs_description/meshes/rear_right_hip.dae" />
+            </geometry>
+        </visual>
+        <collision>
+            <geometry>
+                <mesh filename="package://rs_description/meshes/rear_right_hip_collision.stl" />
+            </geometry>
+        </collision>
+        <inertial>
+            <mass value="0.5" />
+    	    <inertia  ixx="0.01" ixy="0.0"  ixz="0.0"  iyy="0.0"  iyz="0.0"  izz="0.0" />
+    	</inertial>
+    </link>
+    <joint name="rear_right_hip_x" type="revolute">
+        <origin xyz="-0.29785 -0.05500 0.00000" rpy="0 0 0" />
+        <axis xyz="1 0 0" />
+        <parent link="body" />
+        <child link="rear_right_hip" />
+        <dynamics damping="0.0" friction="0.0"/>
+        <limit effort="1000" velocity="1000.00" lower="-0.78539816339744827899" upper="0.78539816339744827899" />
+    </joint>
+    <transmission name="rear_right_hip_x_trans">
+	  <type>transmission_interface/SimpleTransmission</type>
+	  <joint name="rear_right_hip_x">
+          	<hardwareInterface>EffortJointInterface</hardwareInterface>
+          </joint>
+	  <actuator name="rear_right_hip_x">
+          	<mechanicalReduction>50</mechanicalReduction>
+          	<hardwareInterface>EffortJointInterface</hardwareInterface>
+	  </actuator>
+    </transmission>
+<!-- rear_right_upper_leg -->
+    <link name="rear_right_upper_leg">
+        <visual>
+            <geometry>
+                <mesh filename="package://rs_description/meshes/rear_right_upper_leg.dae" />
+            </geometry>
+        </visual>
+        <collision>
+            <geometry>
+                <mesh filename="package://rs_description/meshes/rear_right_upper_leg_collision.stl" />
+            </geometry>
+        </collision>
+        <inertial>
+            <mass value="2.5" />
+    	    <inertia  ixx="0.8" ixy="0.0"  ixz="0.0"  iyy="0.2"  iyz="0.0"  izz="0.0" />
+    	</inertial>
+    </link>
+    <joint name="rear_right_hip_y" type="revolute">
+        <origin xyz="0.0 -0.110945 0.0" rpy="0 0 0" />
+        <axis xyz="0 1 0" />
+        <parent link="rear_right_hip" />
+        <child link="rear_right_upper_leg" />
+        <dynamics damping="0.0" friction="0.0"/>
+        <limit effort="1000" velocity="1000.00" lower="-0.89884456477707963539" upper="2.2951079663725435509" />
+    </joint>
+    <transmission name="rear_right_hip_y_trans">
+	  <type>transmission_interface/SimpleTransmission</type>
+	  <joint name="rear_right_hip_y">
+          	<hardwareInterface>EffortJointInterface</hardwareInterface>
+          </joint>
+	  <actuator name="rear_right_hip_y">
+          	<mechanicalReduction>50</mechanicalReduction>
+          	<hardwareInterface>EffortJointInterface</hardwareInterface>
+	  </actuator>
+    </transmission>
+<!-- rear_right_lower_leg -->
+    <link name="rear_right_lower_leg">
+        <visual>
+            <geometry>
+                <mesh filename="package://rs_description/meshes/rear_right_lower_leg.dae" />
+            </geometry>
+        </visual>
+        <collision>
+            <geometry>
+                <mesh filename="package://rs_description/meshes/rear_right_lower_leg_collision.stl" />
+            </geometry>
+        </collision>
+        <inertial>
+            <mass value="1.5" />
+    	    <inertia  ixx="0.0" ixy="0.0"  ixz="0.0"  iyy="0.125"  iyz="0.0"  izz="0.0" />
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
Commit message: added low level control

File: rs_description/urdf/spot.urdf.xacro (robot description, xacro)
@@ -14,5 +14,5 @@
         </collision>
         <inertial>
-             <mass value="1.25" />
+             <mass value="16.25" />
              <inertia  ixx="0.1" ixy="0.0"  ixz="0.0"  iyy="0.1"  iyz="0.0"  izz="0.077" />
     	</inertial>
@@ -121,5 +121,5 @@
             </geometry>
         </collision>
-        <inertial>
+        <inertial>right
             <mass value="1.5" />
     	    <inertia  ixx="0.0" ixy="0.0"  ixz="0.0"  iyy="0.125"  iyz="0.0"  izz="0.0" />
@@ -459,3 +459,8 @@
 	  </actuator>
     </transmission>
+    <gazebo>
+    	<plugin name="gazebo_ros_control" filename="libgazebo_ros_control.so">
+    	<robotNamespace>/spot</robotNamespace>
+  	</plugin>
+    </gazebo>
 </robot>

Commit message: changed mass of links

File: rs_description/urdf/spot.urdf.xacro (robot description, xacro)
@@ -52,5 +52,5 @@
         </collision>
         <inertial>
-            <mass value="0.5" />
+            <mass value="2.5" />
     	    <inertia  ixx="0.01" ixy="0.0"  ixz="0.0"  iyy="0.0"  iyz="0.0"  izz="0.0" />
     	</inertial>
@@ -87,5 +87,5 @@
         </collision>
         <inertial>
-            <mass value="2.5" />
+            <mass value="1.5" />
     	    <inertia  ixx="0.8" ixy="0.0"  ixz="0.0"  iyy="0.2"  iyz="0.0"  izz="0.0" />
     	</inertial>
@@ -122,5 +122,5 @@
         </collision>
         <inertial>right
-            <mass value="1.5" />
+            <mass value="0.5" />
     	    <inertia  ixx="0.0" ixy="0.0"  ixz="0.0"  iyy="0.125"  iyz="0.0"  izz="0.0" />
     	</inertial>
@@ -157,5 +157,5 @@
         </collision>
         <inertial>
-            <mass value="0.5" />
+            <mass value="2.5" />
     	    <inertia  ixx="0.01" ixy="0.0"  ixz="0.0"  iyy="0.0"  iyz="0.0"  izz="0.0" />
     	</inertial>
@@ -192,5 +192,5 @@
         </collision>
         <inertial>
-            <mass value="2.5" />
+            <mass value="1.5" />
     	    <inertia  ixx="0.8" ixy="0.0"  ixz="0.0"  iyy="0.2"  iyz="0.0"  izz="0.0" />
     	</inertial>
@@ -227,5 +227,5 @@
         </collision>
         <inertial>
-            <mass value="1.5" />
+            <mass value="0.5" />
     	    <inertia  ixx="0.0" ixy="0.0"  ixz="0.0"  iyy="0.125"  iyz="0.0"  izz="0.0" />
     	</inertial>
@@ -262,5 +262,5 @@
         </collision>
         <inertial>
-            <mass value="0.5" />
+            <mass value="2.5" />
     	    <inertia  ixx="0.01" ixy="0.0"  ixz="0.0"  iyy="0.0"  iyz="0.0"  izz="0.0" />
     	</inertial>
@@ -297,5 +297,5 @@
         </collision>
         <inertial>
-           <mass value="2.5" />
+           <mass value="1.5" />
     	   <inertia  ixx="0.8" ixy="0.0"  ixz="0.0"  iyy="0.2"  iyz="0.0"  izz="0.0" />
     	</inertial>
@@ -332,5 +332,5 @@
         </collision>
         <inertial>
-            <mass value="1.5" />
+            <mass value="0.5" />
     	    <inertia  ixx="0.0" ixy="0.0"  ixz="0.0"  iyy="0.125"  iyz="0.0"  izz="0.0" />
     	</inertial>
@@ -367,5 +367,5 @@
         </collision>
         <inertial>
-            <mass value="0.5" />
+            <mass value="2.5" />
     	    <inertia  ixx="0.01" ixy="0.0"  ixz="0.0"  iyy="0.0"  iyz="0.0"  izz="0.0" />
     	</inertial>
@@ -402,5 +402,5 @@
         </collision>
         <inertial>
-            <mass value="2.5" />
+            <mass value="1.5" />
     	    <inertia  ixx="0.8" ixy="0.0"  ixz="0.0"  iyy="0.2"  iyz="0.0"  izz="0.0" />
     	</inertial>
@@ -437,5 +437,5 @@
         </collision>
         <inertial>
-            <mass value="1.5" />
+            <mass value="0.5" />
     	    <inertia  ixx="0.0" ixy="0.0"  ixz="0.0"  iyy="0.125"  iyz="0.0"  izz="0.0" />
     	</inertial>
