Commit message: pid tuned

File: rs_description/urdf/spot.urdf.xacro (robot description, xacro)
@@ -15,5 +15,5 @@
         <inertial>
              <mass value="16.25" />
-             <inertia  ixx="0.1" ixy="0.0"  ixz="0.0"  iyy="0.1"  iyz="0.0"  izz="0.077" />
+             <inertia  ixx="0.677" ixy="0.0"  ixz="0.0"  iyy="1.977"  iyz="0.0"  izz="1.977" />
     	</inertial>
     </link>
@@ -52,6 +52,6 @@
         </collision>
         <inertial>
-            <mass value="2.5" />
-    	    <inertia  ixx="0.01" ixy="0.0"  ixz="0.0"  iyy="0.0"  iyz="0.0"  izz="0.0" />
+            <mass value="1.5" />
+    	    <inertia  ixx="0.5" ixy="0.0"  ixz="0.0"  iyy="0.0"  iyz="0.0"  izz="0.0" />
     	</inertial>
     </link>
@@ -61,5 +61,5 @@
         <parent link="body" />
 	<child link="front_left_hip" />
-	<dynamics damping="0.0" friction="0.0"/>
+	<dynamics damping="0.1" friction="0.1"/>
         <limit effort="1000" velocity="1000.00" lower="-0.78539816339744827899" upper="0.78539816339744827899" />
     </joint>
@@ -88,5 +88,5 @@
         <inertial>
             <mass value="1.5" />
-    	    <inertia  ixx="0.8" ixy="0.0"  ixz="0.0"  iyy="0.2"  iyz="0.0"  izz="0.0" />
+    	    <inertia  ixx="0.0" ixy="0.0"  ixz="0.0"  iyy="0.125"  iyz="0.0"  izz="0.0" />
     	</inertial>
     </link>
@@ -96,5 +96,5 @@
         <parent link="front_left_hip" />
 	<child link="front_left_upper_leg" />
-	<dynamics damping="0.0" friction="0.0"/>
+	<dynamics damping="0.1" friction="0.1"/>
         <limit effort="1000" velocity="1000.00" lower="-0.89884456477707963539" upper="2.2951079663725435509" />
     </joint>
@@ -122,6 +122,6 @@
         </collision>
         <inertial>right
-            <mass value="0.5" />
-    	    <inertia  ixx="0.0" ixy="0.0"  ixz="0.0"  iyy="0.125"  iyz="0.0"  izz="0.0" />
+            <mass value="1.0" />
+    	    <inertia  ixx="0.0" ixy="0.0"  ixz="0.0"  iyy="0.08"  iyz="0.0"  izz="0.0" />
     	</inertial>
     </link>
@@ -131,5 +131,5 @@
         <parent link="front_left_upper_leg" />
         <child link="front_left_lower_leg" />
-        <dynamics damping="0.0" friction="0.0"/>
+        <dynamics damping="0.1" friction="0.1"/>
         <limit effort="1000" velocity="1000.00" lower="-2.7929" upper="-0.254801" />
     </joint>
@@ -157,6 +157,6 @@
         </collision>
         <inertial>
-            <mass value="2.5" />
-    	    <inertia  ixx="0.01" ixy="0.0"  ixz="0.0"  iyy="0.0"  iyz="0.0"  izz="0.0" />
+            <mass value="1.5" />
+    	    <inertia  ixx="0.5" ixy="0.0"  ixz="0.0"  iyy="0.0"  iyz="0.0"  izz="0.0" />
     	</inertial>
     </link>
@@ -166,5 +166,5 @@
         <parent link="body" />
         <child link="front_right_hip" />
-        <dynamics damping="0.0" friction="0.0"/>
+        <dynamics damping="0.1" friction="0.1"/>
         <limit effort="1000" velocity="1000.00" lower="-0.78539816339744827899" upper="0.78539816339744827899" />
     </joint>
@@ -193,5 +193,5 @@
         <inertial>
             <mass value="1.5" />
-    	    <inertia  ixx="0.8" ixy="0.0"  ixz="0.0"  iyy="0.2"  iyz="0.0"  izz="0.0" />
+    	    <inertia  ixx="0.0" ixy="0.0"  ixz="0.0"  iyy="0.125"  iyz="0.0"  izz="0.0" />
     	</inertial>
     </link>
@@ -201,5 +201,5 @@
         <parent link="front_right_hip" />
         <child link="front_right_upper_leg" />
-        <dynamics damping="0.0" friction="0.0"/>
+        <dynamics damping="0.1" friction="0.1"/>
         <limit effort="1000" velocity="1000.00" lower="-0.89884456477707963539" upper="2.2951079663725435509" />
     </joint>
@@ -227,6 +227,6 @@
         </collision>
         <inertial>
-            <mass value="0.5" />
-    	    <inertia  ixx="0.0" ixy="0.0"  ixz="0.0"  iyy="0.125"  iyz="0.0"  izz="0.0" />
+            <mass value="1.0" />
+    	    <inertia  ixx="0.0" ixy="0.0"  ixz="0.0"  iyy="0.08"  iyz="0.0"  izz="0.0" />
     	</inertial>
     </link>
@@ -236,5 +236,5 @@
         <parent link="front_right_upper_leg" />
         <child link="front_right_lower_leg" />
-        <dynamics damping="0.0" friction="0.0"/>
+        <dynamics damping="0.1" friction="0.1"/>
         <limit effort="1000" velocity="1000.00" lower="-2.7929" upper="-0.247563" />
     </joint>
@@ -262,6 +262,6 @@
         </collision>
         <inertial>
-            <mass value="2.5" />
-    	    <inertia  ixx="0.01" ixy="0.0"  ixz="0.0"  iyy="0.0"  iyz="0.0"  izz="0.0" />
+            <mass value="1.5" />
+    	    <inertia  ixx="0.5" ixy="0.0"  ixz="0.0"  iyy="0.0"  iyz="0.0"  izz="0.0" />
     	</inertial>
     </link>
@@ -271,5 +271,5 @@
         <parent link="body" />
         <child link="rear_left_hip" />
-        <dynamics damping="0.0" friction="0.0"/>
+        <dynamics damping="0.1" friction="0.1"/>
         <limit effort="1000" velocity="1000.00" lower="-0.78539816339744827899" upper="0.78539816339744827899" />
     </joint>
@@ -298,5 +298,5 @@
         <inertial>
            <mass value="1.5" />
-    	   <inertia  ixx="0.8" ixy="0.0"  ixz="0.0"  iyy="0.2"  iyz="0.0"  izz="0.0" />
+    	   <inertia  ixx="0.0" ixy="0.0"  ixz="0.0"  iyy="0.125"  iyz="0.0"  izz="0.0" />
     	</inertial>
     </link>
@@ -306,5 +306,5 @@
         <parent link="rear_left_hip" />
         <child link="rear_left_upper_leg" />
-        <dynamics damping="0.0" friction="0.0"/>
+        <dynamics damping="0.1" friction="0.1"/>
         <limit effort="1000" velocity="1000.00" lower="-0.89884456477707963539" upper="2.2951079663725435509" />
     </joint>
@@ -332,6 +332,6 @@
         </collision>
         <inertial>
-            <mass value="0.5" />
-    	    <inertia  ixx="0.0" ixy="0.0"  ixz="0.0"  iyy="0.125"  iyz="0.0"  izz="0.0" />
+            <mass value="1.0" />
+    	    <inertia  ixx="0.0" ixy="0.0"  ixz="0.0"  iyy="0.08"  iyz="0.0"  izz="0.0" />
     	</inertial>
     </link>
@@ -341,5 +341,5 @@
         <parent link="rear_left_upper_leg" />
         <child link="rear_left_lower_leg" />
-        <dynamics damping="0.0" friction="0.0"/>
+        <dynamics damping="0.1" friction="0.1"/>
         <limit effort="1000" velocity="1000.00" lower="-2.7929" upper="-0.267153" />
     </joint>
@@ -367,6 +367,6 @@
         </collision>
         <inertial>
-            <mass value="2.5" />
-    	    <inertia  ixx="0.01" ixy="0.0"  ixz="0.0"  iyy="0.0"  iyz="0.0"  izz="0.0" />
+            <mass value="1.5" />
+    	    <inertia  ixx="0.5" ixy="0.0"  ixz="0.0"  iyy="0.0"  iyz="0.0"  izz="0.0" />
     	</inertial>
     </link>
@@ -376,5 +376,5 @@
         <parent link="body" />
         <child link="rear_right_hip" />
-        <dynamics damping="0.0" friction="0.0"/>
+        <dynamics damping="0.1" friction="0.1"/>
         <limit effort="1000" velocity="1000.00" lower="-0.78539816339744827899" upper="0.78539816339744827899" />
     </joint>
@@ -403,5 +403,5 @@
         <inertial>
             <mass value="1.5" />
-    	    <inertia  ixx="0.8" ixy="0.0"  ixz="0.0"  iyy="0.2"  iyz="0.0"  izz="0.0" />
+    	    <inertia  ixx="0.0" ixy="0.0"  ixz="0.0"  iyy="0.125"  iyz="0.0"  izz="0.0" />
     	</inertial>
     </link>
@@ -411,5 +411,5 @@
         <parent link="rear_right_hip" />
         <child link="rear_right_upper_leg" />
-        <dynamics damping="0.0" friction="0.0"/>
+        <dynamics damping="0.1" friction="0.1"/>
         <limit effort="1000" velocity="1000.00" lower="-0.89884456477707963539" upper="2.2951079663725435509" />
     </joint>
@@ -437,6 +437,6 @@
         </collision>
         <inertial>
-            <mass value="0.5" />
-    	    <inertia  ixx="0.0" ixy="0.0"  ixz="0.0"  iyy="0.125"  iyz="0.0"  izz="0.0" />
+            <mass value="1.0" />
+    	    <inertia  ixx="0.0" ixy="0.0"  ixz="0.0"  iyy="0.08"  iyz="0.0"  izz="0.0" />
     	</inertial>
     </link>
@@ -446,5 +446,5 @@
         <parent link="rear_right_upper_leg" />
         <child link="rear_right_lower_leg" />
-        <dynamics damping="0.0" friction="0.0"/>
+        <dynamics damping="0.1" friction="0.1"/>
         <limit effort="1000" velocity="1000.00" lower="-2.7929" upper="-0.257725" />
     </joint>

Commit message: contact sensor

File: rs_description/urdf/spot.urdf.xacro (robot description, xacro)
@@ -126,4 +126,14 @@
     	</inertial>
     </link>
+    <gazebo reference="front_left_lower_leg">
+      <sensor name="front_left_lower_leg_contact_sensor" type="contact">
+        <collision>
+            <geometry>
+                <mesh filename="package://rs_description/meshes/front_left_lower_leg_collision.stl" />
+            </geometry>
+        </collision>
+        <plugin name="contact" filename="libcontact.so"/>
+      </sensor>
+    </gazebo>
     <joint name="front_left_knee" type="revolute">
         <origin xyz="0.025 0.000 -0.3205" rpy="0 0 0" />

Commit message: contact sensor Bumper and yaw control

File: rs_description/urdf/spot.urdf.xacro (robot description, xacro)
@@ -15,5 +15,5 @@
         <inertial>
              <mass value="16.25" />
-             <inertia  ixx="0.677" ixy="0.0"  ixz="0.0"  iyy="1.977"  iyz="0.0"  izz="1.977" />
+             <inertia  ixx="0.085" ixy="0.0"  ixz="0.0"  iyy="1.045"  iyz="0.0"  izz="1.042" />
     	</inertial>
     </link>
@@ -28,5 +28,5 @@
     <link name="front_rail"/>
     <joint name="front_rail_joint" type="fixed">
-        <origin xyz="0.223 0 0.0805" rpy="0 0 0" />
+        <origin xyz="0.223 0 0.04505" rpy="0 0 0" />
         <parent link="body" />
         <child link="front_rail" />
@@ -35,5 +35,5 @@
     <link name="rear_rail"/>
     <joint name="rear_rail_joint" type="fixed">
-        <origin xyz="-0.223 0 0.0805" rpy="0 0 0" />
+        <origin xyz="-0.223 0 0.04505" rpy="0 0 0" />
         <parent link="body" />
         <child link="rear_rail" />
@@ -53,5 +53,5 @@
         <inertial>
             <mass value="1.5" />
-    	    <inertia  ixx="0.5" ixy="0.0"  ixz="0.0"  iyy="0.0"  iyz="0.0"  izz="0.0" />
+    	    <inertia  ixx="0.0605" ixy="0.0"  ixz="0.0"  iyy="0.0"  iyz="0.0"  izz="0.0" />
     	</inertial>
     </link>
@@ -88,5 +88,5 @@
         <inertial>
             <mass value="1.5" />
-    	    <inertia  ixx="0.0" ixy="0.0"  ixz="0.0"  iyy="0.125"  iyz="0.0"  izz="0.0" />
+    	    <inertia  ixx="0.0" ixy="0.0"  ixz="0.0"  iyy="0.05"  iyz="0.0"  izz="0.0" />
     	</inertial>
     </link>
@@ -116,5 +116,5 @@
             </geometry>
         </visual>
-        <collision>
+        <collision name="front_left_lower_leg_fixed_joint_lump__front_bump_sensor">
             <geometry>
                 <mesh filename="package://rs_description/meshes/front_left_lower_leg_collision.stl" />
@@ -123,17 +123,7 @@
         <inertial>right
             <mass value="1.0" />
-    	    <inertia  ixx="0.0" ixy="0.0"  ixz="0.0"  iyy="0.08"  iyz="0.0"  izz="0.0" />
-    	</inertial>
-    </link>
-    <gazebo reference="front_left_lower_leg">
-      <sensor name="front_left_lower_leg_contact_sensor" type="contact">
-        <collision>
-            <geometry>
-                <mesh filename="package://rs_description/meshes/front_left_lower_leg_collision.stl" />
-            </geometry>
-        </collision>
-        <plugin name="contact" filename="libcontact.so"/>
-      </sensor>
-    </gazebo>
+    	    <inertia  ixx="0.0" ixy="0.0"  ixz="0.0"  iyy="0.045"  iyz="0.0"  izz="0.0" />
+    	</inertial>
+    </link>
     <joint name="front_left_knee" type="revolute">
         <origin xyz="0.025 0.000 -0.3205" rpy="0 0 0" />
@@ -144,4 +134,17 @@
         <limit effort="1000" velocity="1000.00" lower="-2.7929" upper="-0.254801" />
     </joint>
+     <!-- Contact Sensor -->
+  <gazebo reference="front_left_lower_leg">
+    <sensor name="front_left_lower_leg_contactsensor_sensor" type="contact">
+      <always_on>true</always_on>
+      <contact>
+        <collision>front_left_lower_leg_fixed_joint_lump__front_bump_sensor_collision</collision>
+      </contact>
+      <plugin filename="libgazebo_ros_bumper.so" name="front_left_lower_leg_plugin">
+        <bumperTopicName>front_left_lower_leg_contact</bumperTopicName>
+        <frameName>front_left_lower_leg</frameName>
+      </plugin>
+    </sensor>
+  </gazebo>
     <transmission name="front_left_knee_trans">
 	  <type>transmission_interface/SimpleTransmission</type>
@@ -168,5 +171,5 @@
         <inertial>
             <mass value="1.5" />
-    	    <inertia  ixx="0.5" ixy="0.0"  ixz="0.0"  iyy="0.0"  iyz="0.0"  izz="0.0" />
+    	    <inertia  ixx="0.0605" ixy="0.0"  ixz="0.0"  iyy="0.0"  iyz="0.0"  izz="0.0" />
     	</inertial>
     </link>
@@ -203,5 +206,5 @@
         <inertial>
             <mass value="1.5" />
-    	    <inertia  ixx="0.0" ixy="0.0"  ixz="0.0"  iyy="0.125"  iyz="0.0"  izz="0.0" />
+    	    <inertia  ixx="0.0" ixy="0.0"  ixz="0.0"  iyy="0.05"  iyz="0.0"  izz="0.0" />
     	</inertial>
     </link>
@@ -231,5 +234,5 @@
             </geometry>
         </visual>
-        <collision>
+        <collision name="front_right_lower_leg_fixed_joint_lump__front_bump_sensor">
             <geometry>
                 <mesh filename="package://rs_description/meshes/front_right_lower_leg_collision.stl" />
@@ -238,5 +241,5 @@
         <inertial>
             <mass value="1.0" />
-    	    <inertia  ixx="0.0" ixy="0.0"  ixz="0.0"  iyy="0.08"  iyz="0.0"  izz="0.0" />
+    	    <inertia  ixx="0.0" ixy="0.0"  ixz="0.0"  iyy="0.045"  iyz="0.0"  izz="0.0" />
     	</inertial>
     </link>
@@ -249,4 +252,17 @@
         <limit effort="1000" velocity="1000.00" lower="-2.7929" upper="-0.247563" />
     </joint>
+     <!-- Contact Sensor -->
+  <gazebo reference="front_right_lower_leg">
+    <sensor name="front_right_lower_leg_contactsensor_sensor" type="contact">
+      <always_on>true</always_on>
+      <contact>
+        <collision>front_right_lower_leg_fixed_joint_lump__front_bump_sensor_collision</collision>
+      </contact>
+      <plugin filename="libgazebo_ros_bumper.so" name="front_right_lower_leg_plugin">
+        <bumperTopicName>front_right_lower_leg_contact</bumperTopicName>
+        <frameName>front_right_lower_leg</frameName>
+      </plugin>
+    </sensor>
+  </gazebo>
     <transmission name="front_right_knee_trans">
 	  <type>transmission_interface/SimpleTransmission</type>
@@ -273,5 +289,5 @@
         <inertial>
             <mass value="1.5" />
-    	    <inertia  ixx="0.5" ixy="0.0"  ixz="0.0"  iyy="0.0"  iyz="0.0"  izz="0.0" />
+    	    <inertia  ixx="0.0605" ixy="0.0"  ixz="0.0"  iyy="0.0"  iyz="0.0"  izz="0.0" />
     	</inertial>
     </link>
@@ -308,5 +324,5 @@
         <inertial>
            <mass value="1.5" />
-    	   <inertia  ixx="0.0" ixy="0.0"  ixz="0.0"  iyy="0.125"  iyz="0.0"  izz="0.0" />
+    	   <inertia  ixx="0.0" ixy="0.0"  ixz="0.0"  iyy="0.05"  iyz="0.0"  izz="0.0" />
     	</inertial>
     </link>
@@ -336,5 +352,5 @@
             </geometry>
         </visual>
-        <collision>
+        <collision name="rear_left_lower_leg_fixed_joint_lump__rear_bump_sensor">
             <geometry>
                 <mesh filename="package://rs_description/meshes/rear_left_lower_leg_collision.stl" />
@@ -343,5 +359,5 @@
         <inertial>
             <mass value="1.0" />
-    	    <inertia  ixx="0.0" ixy="0.0"  ixz="0.0"  iyy="0.08"  iyz="0.0"  izz="0.0" />
+    	    <inertia  ixx="0.0" ixy="0.0"  ixz="0.0"  iyy="0.045"  iyz="0.0"  izz="0.0" />
     	</inertial>
     </link>
@@ -354,4 +370,17 @@
         <limit effort="1000" velocity="1000.00" lower="-2.7929" upper="-0.267153" />
     </joint>
+     <!-- Contact Sensor -->
+  <gazebo reference="rear_left_lower_leg">
+    <sensor name="rear_left_lower_leg_contactsensor_sensor" type="contact">
+      <always_on>true</always_on>
+      <contact>
+        <collision>rear_left_lower_leg_fixed_joint_lump__rear_bump_sensor_collision</collision>
+      </contact>
+      <plugin filename="libgazebo_ros_bumper.so" name="rear_left_lower_leg_plugin">
+        <bumperTopicName>rear_left_lower_leg_contact</bumperTopicName>
+        <frameName>rear_left_lower_leg</frameName>
+      </plugin>
+    </sensor>
+  </gazebo>
     <transmission name="rear_left_knee_trans">
 	  <type>transmission_interface/SimpleTransmission</type>
@@ -378,5 +407,5 @@
         <inertial>
             <mass value="1.5" />
-    	    <inertia  ixx="0.5" ixy="0.0"  ixz="0.0"  iyy="0.0"  iyz="0.0"  izz="0.0" />
+    	    <inertia  ixx="0.0605" ixy="0.0"  ixz="0.0"  iyy="0.0"  iyz="0.0"  izz="0.0" />
     	</inertial>
     </link>
@@ -413,5 +442,5 @@
         <inertial>
             <mass value="1.5" />
-    	    <inertia  ixx="0.0" ixy="0.0"  ixz="0.0"  iyy="0.125"  iyz="0.0"  izz="0.0" />
+    	    <inertia  ixx="0.0" ixy="0.0"  ixz="0.0"  iyy="0.05"  iyz="0.0"  izz="0.0" />
     	</inertial>
     </link>
@@ -441,5 +470,5 @@
             </geometry>
         </visual>
-        <collision>
+        <collision name='rear_right_lower_leg_fixed_joint_lump__rear_bump_sensor'>
             <geometry>
                 <mesh filename="package://rs_description/meshes/rear_right_lower_leg_collision.stl" />
@@ -448,5 +477,5 @@
         <inertial>
             <mass value="1.0" />
-    	    <inertia  ixx="0.0" ixy="0.0"  ixz="0.0"  iyy="0.08"  iyz="0.0"  izz="0.0" />
+    	    <inertia  ixx="0.0" ixy="0.0"  ixz="0.0"  iyy="0.045"  iyz="0.0"  izz="0.0" />
     	</inertial>
     </link>
@@ -459,4 +488,17 @@
         <limit effort="1000" velocity="1000.00" lower="-2.7929" upper="-0.257725" />
     </joint>
+  <!-- Contact Sensor -->
+  <gazebo reference="rear_right_lower_leg">
+    <sensor name="rear_right_lower_leg_contactsensor_sensor" type="contact">
+      <always_on>true</always_on>
+      <contact>
+        <collision>rear_right_lower_leg_fixed_joint_lump__rear_bump_sensor_collision</collision>
+      </contact>
+      <plugin filename="libgazebo_ros_bumper.so" name="rear_right_lower_leg_plugin">
+        <bumperTopicName>rear_right_lower_leg_contact</bumperTopicName>
+        <frameName>rear_right_lower_leg</frameName>
+      </plugin>
+    </sensor>
+  </gazebo>
     <transmission name="rear_right_knee_trans">
 	  <type>transmission_interface/SimpleTransmission</type>
